File: -PCB-/PMP_2024-25.kicad_pcb (KiCad board)
At the start: 2 copper layers, 123 x 55.5 mm, 49 parts, among them J1 OUT, J2 5V, J3 GND, J4 CALIB, Q1 NPN 2N3904, Q2 NPN 2N3904, Q3 NPN MPSA42, Q4 NPN 2N3904

Commit message: some edits
excel added too
Parts:
- moved L1 0.21 mm to (67.9, 65.0)
Routing:
- net Net-(IO1-DIS): track 41.3 -> 42.0 mm
- net VCC: track 30.3 -> 31.0 mm

Commit message: PCB update
V2
Parts:
- removed Hole (x4): MountingHole_3mm, MountingHole:MountingHole_3mm
- added REF**: MountingHole_2.2mm_M2_DIN965_Pad, MountingHole:MountingHole_2.2mm_M2_DIN965_Pad, F.Cu at (163.8, 149.7)
- added REF**: MountingHole_2.2mm_M2_DIN965_Pad, MountingHole:MountingHole_2.2mm_M2_DIN965_Pad, F.Cu at (129.2, 149.7)
- added REF**: MountingHole_2.2mm_M2_DIN965_Pad, MountingHole:MountingHole_2.2mm_M2_DIN965_Pad, F.Cu at (163.8, 45.1)
- added REF**: MountingHole_2.2mm_M2_DIN965_Pad, MountingHole:MountingHole_2.2mm_M2_DIN965_Pad, F.Cu at (129.3, 45.1)
- J4: value CALIB -> TEST
- R11: footprint Resistor_THT:R_Axial_DIN0207_L6.3mm_D2.5mm_P10.16mm_Horizontal -> Potentiometer_THT:Potentiometer_Bourns_3266W_Vertical
- R14: value ? -> 1k
- moved J4 126.1 mm to (159.4, 149.7), turned to 0 degrees
- moved J2 124.0 mm to (138.4, 149.5), turned to 0 degrees
- moved J3 123.3 mm to (141.0, 149.5), turned to 0 degrees
- moved GC1 123.2 mm to (119.6, 151.2), turned to 90 degrees
- moved J1 117.8 mm to (135.9, 149.5), turned to 0 degrees
- moved R1 106.5 mm to (164.1, 134.9), turned to -90 degrees
- moved C3 105.5 mm to (138.3, 145.0)
- moved R13 102.0 mm to (148.3, 131.8)
- moved R3 102.0 mm to (160.8, 134.9), turned to -90 degrees
- moved R4 97.6 mm to (157.5, 134.9), turned to -90 degrees
- moved R5 93.1 mm to (154.2, 134.9), turned to -90 degrees
- moved L1 92.0 mm to (137.7, 125.1), turned to 90 degrees
- moved R9 91.0 mm to (137.8, 109.3), turned to 90 degrees
- moved R2 90.1 mm to (133.0, 137.3), turned to 90 degrees
- moved R6 88.7 mm to (150.9, 134.9), turned to -90 degrees
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Routing:
- net RES: track 88.1 -> 0.00 mm
- net TRIG: track 62.4 -> 0.00 mm
- net Net-(BZ1-+): track 58.4 -> 0.00 mm
- net CALIB: track 58.1 -> 0.00 mm
- net Net-(IO2-VCC): track 50.1 -> 0.00 mm
- net Net-(IO1-Q): track 44.8 -> 0.00 mm
- net Net-(IO1-DIS): track 42.0 -> 0.00 mm
- net Net-(C5-Pad2): track 40.3 -> 0.00 mm
- net VCC: track 31.0 -> 0.06 mm
- net Net-(Q3-C): track 29.4 -> 0.00 mm
- net Net-(IO2-THR): track 29.0 -> 0.00 mm
- net Net-(D1-K): track 27.6 -> 0.00 mm
- net step_2: track 26.6 -> 0.00 mm
- net step_1: track 21.1 -> 0.00 mm
- net Net-(Q4-B): track 16.1 -> 0.00 mm
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- removed copper zone on B.Cu, net GND
Other:
- board size 123 x 55.5 mm -> 55 x 110 mm

Commit message: more changes
Parts:
- renumbered REF** to Mount1, REF** to Mount2, REF** to Mount3, REF** to Mount4
Changed lines of the file:
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@@
 		(tags "THT DIP DIL PDIP 2.54mm 7.62mm 300mil Socket LongPads")
 		(property "Reference" "IO1"
-			(at 3.81 -2.33 270)
+			(at 3.81 -2.33 -90)
 			(layer "F.SilkS")
 			(effects
@@
 		)
 		(property "Value" "NE555"
-			(at 3.81 9.95 270)
+			(at 3.81 9.95 -90)
 			(layer "F.Fab")
 			(effects
@@
 		)
 		(fp_text user "${REFERENCE}"
-			(at 3.81 3.81 270)
+			(at 3.81 3.81 -90)
 			(layer "F.Fab")
 			(effects
@@
 		(tags "C Disc series Radial pin pitch 5.00mm  diameter 4.3mm width 1.9mm Capacitor")
 		(property "Reference" "C5"
-			(at 2.5 -2.2 360)
+			(at 2.5 -2.2 0)
 			(layer "F.SilkS")
 			(effects
@@
 		)
 		(property "Value" "270pF"
-			(at 2.5 2.2 360)
+			(at 2.5 2.2 0)
 			(layer "F.Fab")
 			(effects
@@
 		)
 		(fp_text user "${REFERENCE}"
-			(at 2.5 0 360)
+			(at 2.5 0 0)
 			(layer "F.Fab")
 			(effects
@@
 		(tags "Through hole pin header THT 1x01 1.00mm single row")
 		(property "Reference" "J3"
-			(at 0 -1.56 360)
+			(at 0 -1.56 0)
 			(layer "F.SilkS")
 			(effects
@@
 		)
 		(property "Value" "GND"
-			(at 0 1.56 360)
+			(at 0 1.56 0)
 			(layer "F.Fab")
 			(effects
@@
 		(tags "C Disc series Radial pin pitch 5.00mm  diameter 4.3mm width 1.9mm Capacitor")
 		(property "Reference" "C1"
-			(at 2.5 -2.2 270)
+			(at 2.5 -2.2 -90)
 			(layer "F.SilkS")
 			(effects
@@
 		)
 		(property "Value" "10nF / 1kV"
-			(at 2.5 2.2 270)
+			(at 2.5 2.2 -90)
 			(layer "F.Fab")
 			(effects
@@
 		)
 		(fp_text user "${REFERENCE}"
-			(at 2.5 0 270)
+			(at 2.5 0 -90)
 			(layer "F.Fab")
 			(effects
@@
 		(tags "C Disc series Radial pin pitch 5.00mm  diameter 4.3mm width 1.9mm Capacitor")
 		(property "Reference" "C4"
-			(at 2.5 -2.2 360)
+			(at 2.5 -2.2 0)
 			(layer "F.SilkS")
 			(effects
@@
 		)
 		(property "Value" "10nF / 1kV"
-			(at 2.5 2.2 360)
+			(at 2.5 2.2 0)
 			(layer "F.Fab")
 			(effects
@@
 		)
 		(fp_text user "${REFERENCE}"
-			(at 2.5 0 360)
+			(at 2.5 0 0)
 			(layer "F.Fab")
 			(effects
@@
 		(tags "Through hole pin header THT 1x01 1.00mm single row")
 		(property "Reference" "J1"
-			(at 0 -1.56 360)
+			(at 0 -1.56 0)
 			(layer "F.SilkS")
 			(effects
@@
 		)
 		(property "Value" "OUT"
-			(at 0 1.56 360)
+			(at 0 1.56 0)
 			(layer "F.Fab")
 			(effects
@@
 		(tags "THT DIP DIL PDIP 2.54mm 7.62mm 300mil Socket LongPads")
 		(property "Reference" "IO2"
-			(at 3.81 -2.33 270)
+			(at 3.81 -2.33 -90)
 			(layer "F.SilkS")
 			(effects
@@
 		)
 		(property "Value" "NE555"
-			(at 3.81 9.95 270)
+			(at 3.81 9.95 -90)
 			(layer "F.Fab")
 			(effects
@@
 		)
 		(fp_text user "${REFERENCE}"
-			(at 3.81 3.81 270)
+			(at 3.81 3.81 -90)
 			(layer "F.Fab")
 			(effects
@@
 		(tags "to-92 sc-43 sc-43a sot54 PA33 transistor")
 		(property "Reference" "Q2"
-			(at 1.27 -3.56 270)
+			(at 1.27 -3.56 -90)
 			(layer "F.SilkS")
 			(effects
@@
 		)
 		(property "Value" "NPN 2N3904"
-			(at 1.27 2.79 270)
+			(at 1.27 2.79 -90)
 			(layer "F.Fab")
 			(effects
@@
 		)
 		(fp_text user "${REFERENCE}"
-			(at 1.27 0 270)
+			(at 1.27 0 -90)
 			(layer "F.Fab")
 			(effects
@@
 		(tags "Resistor Axial_DIN0207 series Axial Horizontal pin pitch 10.16mm 0.25W = 1/4W length 6.3mm diameter 2.5mm")
 		(property "Reference" "R8"
-			(at 5.08 -2.37 270)
+			(at 5.08 -2.37 -90)
 			(layer "F.SilkS")
 			(effects
@@
 		)
 		(property "Value" "470K"
-			(at 5.08 2.37 270)
+			(at 5.08 2.37 -90)
 			(layer "F.Fab")
 			(effects
@@
 		)
 		(fp_text user "${REFERENCE}"
-			(at 5.08 0 270)
+			(at 5.08 0 -90)
 			(layer "F.Fab")
 			(effects
@@
 		(tags "Diode A-405 series Axial Horizontal pin pitch 10.16mm  length 5.2mm diameter 2.7mm")
 		(property "Reference" "D1"
-			(at 5.08 -2.47 270)
+			(at 5.08 -2.47 -90)
 			(layer "F.SilkS")
 			(effects
@@
 		)
 		(property "Value" "1N4937"
-			(at 5.08 2.47 270)
+			(at 5.08 2.47 -90)
 			(layer "F.Fab")
 			(effects
@@
 		)
 		(fp_text user "K"
-			(at 0 -1.9 270)
+			(at 0 -1.9 -90)
 			(layer "F.SilkS")
 			(effects
@@
 		)
 		(fp_text user "${REFERENCE}"
-			(at 5.47 0 270)
+			(at 5.47 0 -90)
 			(layer "F.Fab")
 			(effects
@@
 		)
 		(fp_text user "K"
-			(at 0 -1.9 270)
+			(at 0 -1.9 -90)
 			(layer "F.Fab")
 			(effects
@@
 		(tags "Resistor Axial_DIN0207 series Axial Horizontal pin pitch 10.16mm 0.25W = 1/4W length 6.3mm diameter 2.5mm")
 		(property "Reference" "R9"
-			(at 5.08 -2.37 270)
+			(at 5.08 -2.37 -90)
 			(layer "F.SilkS")
 			(effects
@@
 		)
 		(property "Value" "47K"
-			(at 5.08 2.37 270)
+			(at 5.08 2.37 -90)
 			(layer "F.Fab")
 			(effects
@@
 		)
 		(fp_text user "${REFERENCE}"
-			(at 5.08 0 270)
+			(at 5.08 0 -90)
 			(layer "F.Fab")
 			(effects
@@
 		(tags "Diode A-405 series Axial Horizontal pin pitch 10.16mm  length 5.2mm diameter 2.7mm")
 		(property "Reference" "D3"
-			(at 5.08 -2.47 270)
+			(at 5.08 -2.47 -90)
 			(layer "F.SilkS")
 			(effects
@@
 		)
 		(property "Value" "1N4937"
-			(at 5.08 2.47 270)
+			(at 5.08 2.47 -90)
 			(layer "F.Fab")
 			(effects
@@
 		)
 		(fp_text user "K"
-			(at 0 -1.9 270)
+			(at 0 -1.9 -90)
 			(layer "F.SilkS")
 			(effects
@@
 		)
 		(fp_text user "K"
-			(at 0 -1.9 270)
+			(at 0 -1.9 -90)
 			(layer "F.Fab")
 			(effects
@@
 		)
 		(fp_text user "${REFERENCE}"
-			(at 5.47 0 270)
+			(at 5.47 0 -90)
 			(layer "F.Fab")
 			(effects
@@
 		(tags "to-92 sc-43 sc-43a sot54 PA33 transistor")
 		(property "Reference" "Q3"
-			(at 1.27 -3.56 270)
+			(at 1.27 -3.56 -90)
 			(layer "F.SilkS")
 			(effects
@@
 		)
 		(property "Value" "NPN MPSA42"
-			(at 1.27 2.79 270)
+			(at 1.27 2.79 -90)
 			(layer "F.Fab")
 			(effects
@@
 		)
 		(fp_text user "${REFERENCE}"
-			(at 1.27 0 270)
+			(at 1.27 0 -90)
 			(layer "F.Fab")
 			(effects
@@
 		(tags "LED diameter 5.0mm 2 pins")
 		(property "Reference" "D4"
-			(at 1.27 -3.96 270)
+			(at 1.27 -3.96 -90)
 			(layer "F.SilkS")
 			(effects
@@
 		)
 		(property "Value" "LED RED"
-			(at 1.27 3.96 270)
+			(at 1.27 3.96 -90)
 			(layer "F.Fab")
 			(effects
@@
 		)
 		(fp_text user "${REFERENCE}"
-			(at 1.25 0 270)
+			(at 1.25 0 -90)
 			(layer "F.Fab")
 			(effects
@@
 		(tags "Resistor Axial_DIN0207 series Axial Horizontal pin pitch 10.16mm 0.25W = 1/4W length 6.3mm diameter 2.5mm")
 		(property "Reference" "R2"
-			(at 5.08 -2.37 270)
+			(at 5.08 -2.37 -90)
 			(layer "F.SilkS")
 			(effects
@@
 		)
 		(property "Value" "10M"
-			(at 5.08 2.37 270)
+			(at 5.08 2.37 -90)
 			(layer "F.Fab")
 			(effects
@@
 		)
 		(fp_text user "${REFERENCE}"
-			(at 5.08 0 270)
+			(at 5.08 0 -90)
 			(layer "F.Fab")
 			(effects
@@
 		(descr "Mounting Hole 2.2mm, M2, DIN965")
 		(tags "mounting hole 2.2mm m2 din965")
-		(property "Reference" "REF**"
+		(property "Reference" "Mount4"
 			(at 0 -2.9 0)
 			(layer "F.SilkS")
@@
 		(tags "Inductor Axial series Axial Horizontal pin pitch 12.7mm  length 7mm diameter 3.3mm Fastron MICC")
 		(property "Reference" "L1"
-			(at 6.35 -2.77 270)
+			(at 6.35 -2.77 -90)
 			(layer "F.SilkS")
 			(effects
@@
 		)
 		(property "Value" "100uH"
-			(at 6.35 2.77 270)
+			(at 6.35 2.77 -90)
 			(layer "F.Fab")
 			(effects
@@
 		)
 		(fp_text user "${REFERENCE}"
-			(at 6.35 0 270)
+			(at 6.35 0 -90)
 			(layer "F.Fab")
 			(effects
@@
 		(descr "Mounting Hole 2.2mm, M2, DIN965")
 		(tags "mounting hole 2.2mm m2 din965")
-		(property "Reference" "REF**"
+		(property "Reference" "Mount3"
 			(at 0 -2.9 0)
 			(layer "F.SilkS")
@@
 		(tags "Through hole pin header THT 1x01 1.00mm single row")
 		(property "Reference" "J2"
-			(at 0 -1.56 360)
+			(at 0 -1.56 0)
 			(layer "F.SilkS")
 			(effects
@@
 		)
 		(property "Value" "5V"
-			(at 0 1.56 360)
+			(at 0 1.56 0)
 			(layer "F.Fab")
 			(effects
@@
 		(descr "Mounting Hole 2.2mm, M2, DIN965")
 		(tags "mounting hole 2.2mm m2 din965")
-		(property "Reference" "REF**"
+		(property "Reference" "Mount2"
 			(at 0 -2.9 0)
 			(layer "F.SilkS")
@@
 		(tags "Resistor Axial_DIN0207 series Axial Horizontal pin pitch 10.16mm 0.25W = 1/4W length 6.3mm diameter 2.5mm")
 		(property "Reference" "R10"
-			(at 5.08 -2.37 270)
+			(at 5.08 -2.37 -90)
 			(layer "F.SilkS")
 			(effects
@@
 		)
 		(property "Value" "470K"
-			(at 5.08 2.37 270)
+			(at 5.08 2.37 -90)
 			(layer "F.Fab")
 			(effects
@@
 		)
 		(fp_text user "${REFERENCE}"
-			(at 5.08 0 270)
+			(at 5.08 0 -90)
 			(layer "F.Fab")
 			(effects
@@
 		(descr "Mounting Hole 2.2mm, M2, DIN965")
 		(tags "mounting hole 2.2mm m2 din965")
-		(property "Reference" "REF**"
+		(property "Reference" "Mount1"
 			(at 0 -2.9 0)
 			(layer "F.SilkS")

Commit message: PCB pre-final
full pcb design V2 - will add picture on the pcb soon
Parts:
- moved Mount2 4.97 mm to (168.8, 45.1)
- moved Mount4 4.97 mm to (168.8, 149.7)
- moved J4 4.70 mm to (164.1, 149.7)
- moved R6 3.56 mm to (147.3, 134.9)
- moved Q2 2.07 mm to (154.3, 113.8), turned to 0 degrees
- moved R5 1.65 mm to (152.5, 134.9)
- moved R15 0.89 mm to (141.0, 104.3)
- moved R14 0.89 mm to (141.0, 101.1)
- moved C3 0.12 mm to (138.4, 145.1), turned to 90 degrees
Routing:
- net step_1: track 0.00 -> 82.1 mm
- net Net-(IO2-VCC): track 0.00 -> 72.3 mm
- net VCC: track 0.06 -> 62.1 mm
- net TRIG: track 0.00 -> 59.8 mm
- net CALIB: track 0.00 -> 58.2 mm
- net Net-(BZ1-+): track 0.00 -> 52.8 mm
- net Net-(C5-Pad2): track 0.00 -> 45.8 mm
- net Net-(Q1-B): track 0.00 -> 42.1 mm
- net step_2: track 0.00 -> 39.9 mm
- net Net-(Q2-B): track 0.00 -> 27.8 mm
- net RES: track 0.00 -> 25.3 mm
- net Net-(Q4-B): track 0.00 -> 25.1 mm
- net Net-(IO2-THR): track 0.00 -> 23.7 mm
- net Net-(D2-K): track 0.00 -> 18.8 mm
- net Net-(D1-K): track 0.00 -> 18.6 mm
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- added copper zone on B.Cu, net GND
Other:
- board size 55 x 110 mm -> 60 x 110 mm

Commit message: added image on PCB
PDF prints added too
Parts:
- added TP1: TestPoint, graphics:obrazek1, B.Cu at (148.1, 56.1)

Commit message: EDITS ON CHEMATIC AND PCB
renamed pins and changed positions
Parts:
- renumbered J2 to J1, J3 to J2, J1 to J3
Changed lines of the file:
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@@
 		)
 		(property ki_fp_filters "DIP*W7.62mm*")
-		(sheetname "Hlavní")
+		(sheetname "Root")
 		(sheetfile "PMP_2024-25.kicad_sch")
 		(attr through_hole)
@@
 		)
 		(property ki_fp_filters "CP_*")
-		(sheetname "Hlavní")
+		(sheetname "Root")
 		(sheetfile "PMP_2024-25.kicad_sch")
 		(attr through_hole)
@@
 		)
 		(property ki_fp_filters "C_*")
-		(sheetname "Hlavní")
+		(sheetname "Root")
 		(sheetfile "PMP_2024-25.kicad_sch")
 		(attr through_hole)
@@
 		)
 		(property ki_fp_filters "R_*")
-		(sheetname "Hlavní")
+		(sheetname "Root")
 		(sheetfile "PMP_2024-25.kicad_sch")
 		(attr through_hole)
@@
 		(descr "Through hole straight pin header, 1x01, 1.00mm pitch, single row")
 		(tags "Through hole pin header THT 1x01 1.00mm single row")
-		(property "Reference" "J3"
+		(property "Reference" "J2"
 			(at 0 -1.56 0)
 			(layer "F.SilkS")
@@
 		)
 		(property ki_fp_filters "Connector*:*_1x??_*")
-		(sheetname "Hlavní")
+		(sheetname "Root")
 		(sheetfile "PMP_2024-25.kicad_sch")
 		(attr through_hole)
@@
 		)
 		(property ki_fp_filters "C_*")
-		(sheetname "Hlavní")
+		(sheetname "Root")
 		(sheetfile "PMP_2024-25.kicad_sch")
 		(attr through_hole)
@@
 		)
 		(property ki_fp_filters "*Buzzer*")
-		(sheetname "Hlavní")
+		(sheetname "Root")
 		(sheetfile "PMP_2024-25.kicad_sch")
 		(attr through_hole)
@@
 		)
 		(property ki_fp_filters "R_*")
-		(sheetname "Hlavní")
+		(sheetname "Root")
 		(sheetfile "PMP_2024-25.kicad_sch")
 		(attr through_hole)
@@
 		)
 		(property ki_fp_filters "CP_*")
-		(sheetname "Hlavní")
+		(sheetname "Root")
 		(sheetfile "PMP_2024-25.kicad_sch")
 		(attr through_hole)
@@
 		)
 		(property ki_fp_filters "C_*")
-		(sheetname "Hlavní")
+		(sheetname "Root")
 		(sheetfile "PMP_2024-25.kicad_sch")
 		(attr through_hole)
@@
 		)
 		(property ki_fp_filters "C_*")
-		(sheetname "Hlavní")
+		(sheetname "Root")
 		(sheetfile "PMP_2024-25.kicad_sch")
 		(attr through_hole)
@@
 		)
 		(property ki_fp_filters "R_*")
-		(sheetname "Hlavní")
+		(sheetname "Root")
 		(sheetfile "PMP_2024-25.kicad_sch")
 		(attr through_hole)
@@
 		)
 		(property ki_fp_filters "C_*")
-		(sheetname "Hlavní")
+		(sheetname "Root")
 		(sheetfile "PMP_2024-25.kicad_sch")
 		(attr through_hole)
@@
 		(descr "Through hole straight pin header, 1x01, 1.00mm pitch, single row")
 		(tags "Through hole pin header THT 1x01 1.00mm single row")
-		(property "Reference" "J1"
+		(property "Reference" "J3"
 			(at 0 -1.56 0)
 			(layer "F.SilkS")
@@
 		)
 		(property ki_fp_filters "Connector*:*_1x??_*")
-		(sheetname "Hlavní")
+		(sheetname "Root")
 		(sheetfile "PMP_2024-25.kicad_sch")
 		(attr through_hole)
@@
 		)
 		(property ki_fp_filters "R_*")
-		(sheetname "Hlavní")
+		(sheetname "Root")
 		(sheetfile "PMP_2024-25.kicad_sch")
 		(attr through_hole)
@@
 			)
 		)
-		(sheetname "Hlavní")
+		(sheetname "Root")
 		(sheetfile "PMP_2024-25.kicad_sch")
 		(attr through_hole)
@@
 		)
 		(property ki_fp_filters "TO-???* *_Diode_* *SingleDiode* D_*")
-		(sheetname "Hlavní")
+		(sheetname "Root")
 		(sheetfile "PMP_2024-25.kicad_sch")
 		(attr through_hole)
@@
 		)
 		(property ki_fp_filters "DIP*W7.62mm*")
-		(sheetname "Hlavní")
+		(sheetname "Root")
 		(sheetfile "PMP_2024-25.kicad_sch")
 		(attr through_hole)
@@
 		)
 		(property ki_fp_filters "R_*")
-		(sheetname "Hlavní")
+		(sheetname "Root")
 		(sheetfile "PMP_2024-25.kicad_sch")
 		(attr through_hole)
@@
 			)
 		)
-		(sheetname "Hlavní")
+		(sheetname "Root")
 		(sheetfile "PMP_2024-25.kicad_sch")
 		(attr through_hole)
@@
 		)
 		(property ki_fp_filters "R_*")
-		(sheetname "Hlavní")
+		(sheetname "Root")
 		(sheetfile "PMP_2024-25.kicad_sch")
 		(attr through_hole)
@@
 		)
 		(property ki_fp_filters "R_*")
-		(sheetname "Hlavní")
+		(sheetname "Root")
 		(sheetfile "PMP_2024-25.kicad_sch")
 		(attr through_hole)
@@
 		)
 		(property ki_fp_filters "Choke_* *Coil* Inductor_* L_*")
-		(sheetname "Hlavní")
+		(sheetname "Root")
 		(sheetfile "PMP_2024-25.kicad_sch")
 		(attr through_hole)
@@
 		)
 		(property ki_fp_filters "TO-???* *_Diode_* *SingleDiode* D_*")
-		(sheetname "Hlavní")
+		(sheetname "Root")
 		(sheetfile "PMP_2024-25.kicad_sch")
 		(attr through_hole)
@@
 		)
 		(property ki_fp_filters "R_*")
-		(sheetname "Hlavní")
+		(sheetname "Root")
 		(sheetfile "PMP_2024-25.kicad_sch")
 		(attr through_hole)
@@
 		)
 		(property ki_fp_filters "Potentiometer*")
-		(sheetname "Hlavní")
+		(sheetname "Root")
 		(sheetfile "PMP_2024-25.kicad_sch")
 		(attr through_hole)
@@
 		)
 		(property ki_fp_filters "TO-???* *_Diode_* *SingleDiode* D_*")
-		(sheetname "Hlavní")
+		(sheetname "Root")
 		(sheetfile "PMP_2024-25.kicad_sch")
 		(attr through_hole)
@@
 			)
 		)
-		(sheetname "Hlavní")
+		(sheetname "Root")
 		(sheetfile "PMP_2024-25.kicad_sch")
 		(attr through_hole)
@@
 		)
 		(property ki_fp_filters "LED* LED_SMD:* LED_THT:*")
-		(sheetname "Hlavní")
+		(sheetname "Root")
 		(sheetfile "PMP_2024-25.kicad_sch")
 		(attr through_hole)
@@
 		)
 		(property ki_fp_filters "R_*")
-		(sheetname "Hlavní")
+		(sheetname "Root")
 		(sheetfile "PMP_2024-25.kicad_sch")
 		(attr through_hole)
@@
 		)
 		(property ki_fp_filters "R_*")
-		(sheetname "Hlavní")
+		(sheetname "Root")
 		(sheetfile "PMP_2024-25.kicad_sch")
 		(attr through_hole)
@@
 		)
 		(property ki_fp_filters "C_*")
-		(sheetname "Hlavní")
+		(sheetname "Root")
 		(sheetfile "PMP_2024-25.kicad_sch")
 		(attr through_hole)
@@
 		)
 		(property ki_fp_filters "C_*")
-		(sheetname "Hlavní")
+		(sheetname "Root")
 		(sheetfile "PMP_2024-25.kicad_sch")
 		(attr through_hole)
@@
 		)
 		(property ki_fp_filters "R_*")
-		(sheetname "Hlavní")
+		(sheetname "Root")
 		(sheetfile "PMP_2024-25.kicad_sch")
 		(attr through_hole)
@@
 		)
 		(property ki_fp_filters "R_*")
-		(sheetname "Hlavní")
+		(sheetname "Root")
 		(sheetfile "PMP_2024-25.kicad_sch")
 		(attr through_hole)
@@
 		)
 		(property ki_fp_filters "Choke_* *Coil* Inductor_* L_*")
-		(sheetname "Hlavní")
+		(sheetname "Root")
 		(sheetfile "PMP_2024-25.kicad_sch")
 		(attr through_hole)
@@
 			)
 		)
-		(sheetname "Hlavní")
+		(sheetname "Root")
 		(sheetfile "PMP_2024-25.kicad_sch")
 		(attr through_hole)
@@
 			)
 		)
-		(sheetname "Hlavní")
+		(sheetname "Root")
 		(sheetfile "PMP_2024-25.kicad_sch")
 		(attr through_hole)
@@
 		)
 		(property ki_fp_filters "Connector*:*_1x??_*")
-		(sheetname "Hlavní")
+		(sheetname "Root")
 		(sheetfile "PMP_2024-25.kicad_sch")
 		(attr through_hole)
@@
 		(descr "Through hole straight pin header, 1x01, 1.00mm pitch, single row")
 		(tags "Through hole pin header THT 1x01 1.00mm single row")
-		(property "Reference" "J2"
+		(property "Reference" "J1"
 			(at 0 -1.56 0)
 			(layer "F.SilkS")
@@
 		)
 		(property ki_fp_filters "Connector*:*_1x??_*")
-		(sheetname "Hlavní")
+		(sheetname "Root")
 		(sheetfile "PMP_2024-25.kicad_sch")
 		(attr through_hole)
@@
 		)
 		(property ki_fp_filters "R_*")
-		(sheetname "Hlavní")
+		(sheetname "Root")
 		(sheetfile "PMP_2024-25.kicad_sch")
 		(attr through_hole)
@@
 		)
 		(property ki_fp_filters "R_*")
-		(sheetname "Hlavní")
+		(sheetname "Root")
 		(sheetfile "PMP_2024-25.kicad_sch")
 		(attr through_hole)
@@
 		)
 		(property ki_fp_filters "R_*")
-		(sheetname "Hlavní")
+		(sheetname "Root")
 		(sheetfile "PMP_2024-25.kicad_sch")
 		(attr through_hole)
@@
 		)
 		(property ki_fp_filters "C_*")
-		(sheetname "Hlavní")
+		(sheetname "Root")
 		(sheetfile "PMP_2024-25.kicad_sch")
 		(attr through_hole)
@@
 		)
 		(property ki_fp_filters "R_*")
-		(sheetname "Hlavní")
+		(sheetname "Root")
 		(sheetfile "PMP_2024-25.kicad_sch")
 		(attr through_hole)
@@
 			)
 		)
+		(property ki_fp_filters "Pin* Test*")
+		(sheetname "Root")
+		(sheetfile "PMP_2024-25.kicad_sch")
 		(attr board_only exclude_from_pos_files)
 		(fp_poly
@@
 		(layer "Dwgs.User")
 		(pts
-			(xy 112.4 152.4) (xy 124.9 152.4)
+			(xy 112.6 149.5) (xy 125.1 149.5)
 		)
 		(height 13.7)
 		(gr_text "12.5 mm"
-			(at 118.65 164.95 0)
+			(at 118.9 161.9 0)
 			(layer "Dwgs.User")
 			(effects
@@
 			(thickness 0.1)
 			(arrow_length 1.27)
-			(text_position_mode 0)
+			(text_position_mode 2)
 			(extension_height 0.58642)
 			(extension_offset 0.5) keep_text_aligned)

Commit message: edits on pcb, design etc.
box model soon, tommorow creating pcb v2
Parts:
- R11: footprint Potentiometer_THT:Potentiometer_Bourns_3266W_Vertical -> Potentiometer_THT:Potentiometer_Bourns_3296W_Vertical
- moved TP1 86.8 mm to (147.1, 142.8), turned to 0 degrees
- moved Q2 24.2 mm to (155.5, 89.6), turned to 90 degrees
- moved R11 22.9 mm to (160.2, 91.2)
- moved R6 22.4 mm to (144.9, 112.6)
- moved C3 22.3 mm to (138.4, 122.8)
- moved C4 22.3 mm to (128.9, 80.2)
- moved IO1 22.3 mm to (143.3, 74.2)
- moved J1 22.3 mm to (138.4, 127.2)
- moved J2 22.3 mm to (141.0, 127.2)
- moved J3 22.3 mm to (135.9, 127.2)
- moved Q3 22.3 mm to (163.3, 109.0)
- moved R10 22.3 mm to (139.4, 73.6)
- moved R2 22.3 mm to (133.0, 115.0)
- moved R8 22.3 mm to (143.4, 60.0)
- moved BZ1 22.3 mm to (151.7, 57.5)
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Connections:
- Mount1 pad 1: (no net) -> GND
- Mount2 pad 1: (no net) -> GND
- Mount3 pad 1: (no net) -> GND
- Mount4 pad 1: (no net) -> GND
Routing:
- net CALIB: track 58.2 -> 66.5 mm
- net Net-(Q2-B): track 27.8 -> 33.2 mm
- net Net-(R5-Pad2): track 5.21 -> 7.65 mm
- net RES: track 25.3 -> 27.1 mm
- net Net-(IO2-VCC): track 72.3 -> 71.8 mm
- net Net-(C5-Pad2): track 45.8 -> 45.3 mm
Other:
- board text added: "GM TUBE SLOT"
- board text added: "Ondřej Kautský PMP"

Commit message: text edits
+export
Parts:
- moved TP1 0.52 mm to (147.5, 142.5)
Other:
- board text added: "+5V"
- board text added: "Controler + Display slot"
- board text added: "GND"
- board text added: "OUT"
- board text added: "TEST"
