File: -PCB-/PMP_2024-25.kicad_pcb (KiCad board)
At the start: 2 copper layers, 60 x 110 mm, 50 parts, among them J1 5V, J2 GND, J3 OUT, J4 TEST, Q1 NPN 2N3904, Q2 NPN 2N3904, Q3 NPN MPSA42, Q4 NPN 2N3904

Commit message: presentation update
Parts:
- moved TP1 135.7 mm to (44.8, 53.8), turned to 180 degrees
